File: Detector_Radio_With_Optional_Amp.kicad_sch (KiCad schematic)
At the start: 19 parts, among them Q1 BC547

Commit message: schematics added
Parts:
- added Rant: 200, symbol Device:R
- Cant1: renamed from Cparasitic; value 270p -> 281p
- gave numbers to parts that had none: 1
- renumbered Ls to Ls3
Connections:
- net GND: no longer Cant1.2
- net at C1.1, Ls3.4: now also Cant1.2; no longer AE1.1 (A), Cant1.1
- new net: AE1.1 (A), Rant.1
- new net: Cant1.1, Rant.2
Other:
- moved on the sheet: AE1, C1, Cant1
